File: pcb/AlarmClock.kicad_sch (KiCad schematic)
At the start: 12 parts, among them J1 Conn_01x08_Pin, SW1 SW_Push, SW2 SW_Push, SW3 SW_Push, SW4 SW_Push, SW5 RotaryEncoder_Switch, U1 XIAO-ESP32-C3-SMD

Commit message: some updates to schem file
Other:
- note added: "connecter pins for display"
- note added: "esp32, switches & buzzer"
- note added: "mounting holes"
- note added: "rotary encoder"
- moved on the sheet: J1, SW5
Changed lines of the file:
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@@
 	(generator_version "10.0")
 	(paper "A4")
+	(rectangle
+		(start 68.58 60.96)
+		(end 185.42 128.27)
+		(stroke
+			(width 0)
+			(type default)
+		)
+		(fill
+			(type none)
+		)
+	)
+	(rectangle
+		(start 187.96 116.84)
+		(end 217.17 147.32)
+		(stroke
+			(width 0)
+			(type default)
+		)
+		(fill
+			(type none)
+		)
+	)
+	(rectangle
+		(start 85.09 129.54)
+		(end 121.92 147.32)
+		(stroke
+			(width 0)
+			(type default)
+		)
+		(fill
+			(type none)
+		)
+	)
+	(rectangle
+		(start 204.47 76.2)
+		(end 228.6 110.49)
+		(stroke
+			(width 0)
+			(type default)
+		)
+		(fill
+			(type none)
+		)
+	)
+	(text "esp32, switches & buzzer\n"
+		(exclude_from_sim no)
+		(at 81.026 59.436 0)
+		(effects
+			(font
+				(size 1.27 1.27)
+			)
+		)
+	)
+	(text "mounting holes\n"
+		(exclude_from_sim no)
+		(at 211.328 74.93 0)
+		(effects
+			(font
+				(size 1.27 1.27)
+			)
+		)
+	)
+	(text "connecter pins for display\n"
+		(exclude_from_sim no)
+		(at 200.406 115.824 0)
+		(effects
+			(font
+				(size 1.27 1.27)
+			)
+		)
+	)
+	(text "rotary encoder\n"
+		(exclude_from_sim no)
+		(at 129.286 131.318 0)
+		(effects
+			(font
+				(size 1.27 1.27)
+			)
+		)
+	)
 	(junction
 		(at 148.59 91.44)
@@
 	(wire
 		(pts
-			(xy 166.37 82.55) (xy 171.45 82.55)
+			(xy 200.66 127) (xy 205.74 127)
 		)
 		(stroke
@@
 	(wire
 		(pts
-			(xy 171.45 82.55) (xy 171.45 73.66)
+			(xy 205.74 127) (xy 205.74 118.11)
 		)
 		(stroke
@@
 	(wire
 		(pts
-			(xy 92.71 134.62) (xy 95.25 134.62)
-		)
-		(stroke
-			(width 0)
-			(type default)
-		)
-	)
-	(wire
-		(pts
-			(xy 168.91 100.33) (xy 166.37 100.33)
-		)
-		(stroke
-			(width 0)
-			(type default)
-		)
-	)
-	(wire
-		(pts
-			(xy 92.71 139.7) (xy 95.25 139.7)
+			(xy 92.71 138.43) (xy 95.25 138.43)
+		)
+		(stroke
+			(width 0)
+			(type default)
+		)
+	)
+	(wire
+		(pts
+			(xy 203.2 144.78) (xy 200.66 144.78)
+		)
+		(stroke
+			(width 0)
+			(type default)
+		)
+	)
+	(wire
+		(pts
+			(xy 92.71 143.51) (xy 95.25 143.51)
 		)
 		(stroke
@@
 	(wire
 		(pts
-			(xy 110.49 134.62) (xy 114.3 134.62)
+			(xy 110.49 138.43) (xy 114.3 138.43)
 		)
 		(stroke
@@
 	(wire
 		(pts
-			(xy 166.37 85.09) (xy 180.34 85.09)
+			(xy 200.66 129.54) (xy 214.63 129.54)
 		)
 		(stroke
@@
 	(wire
 		(pts
-			(xy 171.45 73.66) (xy 175.26 73.66)
+			(xy 205.74 118.11) (xy 209.55 118.11)
 		)
 		(stroke
@@
 	)
 	(label "DC"
-		(at 166.37 95.25 0)
+		(at 200.66 139.7 0)
 		(effects
 			(font
@@
 	)
 	(label "BL"
-		(at 168.91 100.33 180)
+		(at 203.2 144.78 180)
 		(effects
 			(font
@@
 	)
 	(label "B"
-		(at 92.71 139.7 0)
+		(at 92.71 143.51 0)
 		(effects
 			(font
@@
 	)
 	(label "SCL"
-		(at 166.37 87.63 0)
+		(at 200.66 132.08 0)
 		(effects
 			(font
@@
 	)
 	(label "CS"
-		(at 166.37 97.79 0)
+		(at 200.66 142.24 0)
 		(effects
 			(font
@@
 	)
 	(label "A"
-		(at 92.71 134.62 0)
+		(at 92.71 138.43 0)
 		(effects
 			(font
@@
 	)
 	(label "RST"
-		(at 166.37 92.71 0)
+		(at 200.66 137.16 0)
 		(effects
 			(font
@@
 	)
 	(label "SW"
-		(at 114.3 134.62 0)
+		(at 114.3 138.43 0)
 		(effects
 			(font
@@
 	)
 	(label "SDA"
-		(at 166.37 90.17 0)
+		(at 200.66 134.62 0)
 		(effects
 			(font
@@
 	(symbol
 		(lib_id "power:GND")
-		(at 175.26 73.66 0)
+		(at 209.55 118.11 0)
 		(unit 1)
 		(body_style 1)
@@
 		(fields_autoplaced yes)
 		(property "Reference" "#PWR07"
-			(at 175.26 80.01 0)
+			(at 209.55 124.46 0)
 			(hide yes)
 			(show_name no)
@@
 		)
 		(property "Value" "GND"
-			(at 175.26 78.74 0)
+			(at 209.55 123.19 0)
 			(show_name no)
 			(do_not_autoplace no)
@@
 		)
 		(property "Footprint" ""
-			(at 175.26 73.66 0)
+			(at 209.55 118.11 0)
 			(hide yes)
 			(show_name no)
@@
 		)
 		(property "Datasheet" ""
-			(at 175.26 73.66 0)
+			(at 209.55 118.11 0)
 			(hide yes)
 			(show_name no)
@@
 		)
 		(property "Description" "Power symbol creates a global label with name \"GND\" , ground"
-			(at 175.26 73.66 0)
+			(at 209.55 118.11 0)
 			(hide yes)
 			(show_name no)
@@
 	(symbol
 		(lib_id "Connector:Conn_01x08_Pin")
-		(at 161.29 90.17 0)
+		(at 195.58 134.62 0)
 		(unit 1)
 		(body_style 1)
@@
 		(fields_autoplaced yes)
 		(property "Reference" "J1"
-			(at 161.925 77.47 0)
+			(at 196.215 121.92 0)
 			(show_name no)
 			(do_not_autoplace no)
@@
 		)
 		(property "Value" "Conn_01x08_Pin"
-			(at 161.925 80.01 0)
+			(at 196.215 124.46 0)
 			(show_name no)
 			(do_not_autoplace no)
@@
 		)
 		(property "Footprint" "Connector_PinSocket_2.54mm:PinSocket_1x08_P2.54mm_Vertical"
-			(at 161.29 90.17 0)
+			(at 195.58 134.62 0)
 			(hide yes)
 			(show_name no)
@@
 		)
 		(property "Datasheet" ""
-			(at 161.29 90.17 0)
+			(at 195.58 134.62 0)
 			(hide yes)
 			(show_name no)
@@
 		)
 		(property "Description" "Generic connector, single row, 01x08, script generated"
-			(at 161.29 90.17 0)
+			(at 195.58 134.62 0)
 			(hide yes)
 			(show_name no)
@@
 	(symbol
 		(lib_id "power:GND")
-		(at 95.25 137.16 270)
+		(at 95.25 140.97 270)
 		(unit 1)
 		(body_style 1)
@@
 		(fields_autoplaced yes)
 		(property "Reference" "#PWR09"
-			(at 88.9 137.16 0)
+			(at 88.9 140.97 0)
 			(hide yes)
 			(show_name no)
@@
 		)
 		(property "Value" "GND"
-			(at 91.44 137.1599 90)
+			(at 91.44 140.9699 90)
 			(show_name no)
 			(do_not_autoplace no)
@@
 		)
 		(property "Footprint" ""
-			(at 95.25 137.16 0)
+			(at 95.25 140.97 0)
 			(hide yes)
 			(show_name no)
@@
 		)
 		(property "Datasheet" ""
-			(at 95.25 137.16 0)
+			(at 95.25 140.97 0)
 			(hide yes)
 			(show_name no)
@@
 		)
 		(property "Description" "Power symbol creates a global label with name \"GND\" , ground"
-			(at 95.25 137.16 0)
+			(at 95.25 140.97 0)
 			(hide yes)
 			(show_name no)
@@
 	(symbol
 		(lib_id "power:GND")
-		(at 110.49 139.7 90)
+		(at 110.49 143.51 90)
 		(unit 1)
 		(body_style 1)
@@
 		(fields_autoplaced yes)
 		(property "Reference" "#PWR010"
-			(at 116.84 139.7 0)
+			(at 116.84 143.51 0)
 			(hide yes)
 			(show_name no)
@@
 		)
 		(property "Value" "GND"
-			(at 114.3 139.6999 90)
+			(at 114.3 143.5099 90)
 			(show_name no)
 			(do_not_autoplace no)
@@
 		)
 		(property "Footprint" ""
-			(at 110.49 139.7 0)
+			(at 110.49 143.51 0)
 			(hide yes)
 			(show_name no)
@@
 		)
 		(property "Datasheet" ""
-			(at 110.49 139.7 0)
+			(at 110.49 143.51 0)
 			(hide yes)
 			(show_name no)
@@
 		)
 		(property "Description" "Power symbol creates a global label with name \"GND\" , ground"
-			(at 110.49 139.7 0)
+			(at 110.49 143.51 0)
 			(hide yes)
 			(show_name no)
@@
 	(symbol
 		(lib_id "power:+3.3V")
-		(at 180.34 85.09 0)
+		(at 214.63 129.54 0)
 		(unit 1)
 		(body_style 1)
@@
 		(fields_autoplaced yes)
 		(property "Reference" "#PWR08"
-			(at 180.34 88.9 0)
+			(at 214.63 133.35 0)
 			(hide yes)
 			(show_name no)
@@
 		)
 		(property "Value" "+3.3V"
-			(at 180.34 80.01 0)
+			(at 214.63 124.46 0)
 			(show_name no)
 			(do_not_autoplace no)
@@
 		)
 		(property "Footprint" ""
-			(at 180.34 85.09 0)
+			(at 214.63 129.54 0)
 			(hide yes)
 			(show_name no)
@@
 		)
 		(property "Datasheet" ""
-			(at 180.34 85.09 0)
+			(at 214.63 129.54 0)
 			(hide yes)
 			(show_name no)
@@
 		)
 		(property "Description" "Power symbol creates a global label with name \"+3.3V\""
-			(at 180.34 85.09 0)
+			(at 214.63 129.54 0)
 			(hide yes)
 			(show_name no)
@@
 	(symbol
 		(lib_id "Device:RotaryEncoder_Switch")
-		(at 102.87 137.16 0)
+		(at 102.87 140.97 0)
 		(unit 1)
 		(body_style 1)
@@
 		(fields_autoplaced yes)
 		(property "Reference" "SW5"
-			(at 102.87 127 0)
+			(at 102.87 130.81 0)
 			(show_name no)
 			(do_not_autoplace no)
@@
 		)
 		(property "Value" "RotaryEncoder_Switch"
-			(at 102.87 129.54 0)
+			(at 102.87 133.35 0)
 			(show_name no)
 			(do_not_autoplace no)
@@
 		)
 		(property "Footprint" "Rotary_Encoder:RotaryEncoder_Alps_EC11E-Switch_Vertical_H20mm"
-			(at 99.06 133.096 0)
+			(at 99.06 136.906 0)
 			(hide yes)
 			(show_name no)
@@
 		)
 		(property "Datasheet" ""
-			(at 102.87 130.556 0)
+			(at 102.87 134.366 0)
 			(hide yes)
 			(show_name no)
@@
 		)
 		(property "Description" "Rotary encoder, dual channel, incremental quadrate outputs, with switch"
-			(at 102.87 137.16 0)
-			(hide yes)
-			(show_name no)
+			(at 102.87 140.97 0)
+			(hide yes)
+			(show_name no)
